Commit message: dev

File: description/indy7.urdf (robot description, URDF)
Before this commit: robot indy, 9 links, 8 joints
Links:
- link tcp: mass None -> 0.0
Joints:
- joint tcp: origin xyz=0.0                          0.0                          0.06 rpy=0.0                         0.0                         0.0 -> xyz=0 0 0.06 rpy=0 0 0
